File: Air Bearing PCB/Air_Bearing_PCB.kicad_pcb (KiCad board)
At the start: 2 copper layers, 68.6 x 53.3 mm, 21 parts, among them J1 Conn_01x03_Female, J2 Conn_01x02_Female, J3 Conn_01x06_Female, P1 Power, P2 Analog, P3 Digital, P4 Digital, P5 CONN_01X01, P6 CONN_01X01, P7 CONN_01X01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

Commit message: Added Gerber Files
Made a few small routing and schematic edits. Added Gerber files.
Connections:
- P3 pad 1: /A5(SCL) -> /A5(SCL)(2)
- P3 pad 2: /A4(SDA) -> /A4(SDA)(2)
- R1 pad 2: /A4(SDA) -> /A4(SDA)(2)
- R2 pad 2: /A5(SCL) -> /A5(SCL)(2)
- U2 pad 11: /A4(SDA) -> /A4(SDA)(2)
- U2 pad 12: /A5(SCL) -> /A5(SCL)(2)
Routing:
- net /A4(SDA)(2): track 0.00 -> 7.69 mm
- net /A4(SDA): track 7.69 -> 0.00 mm
- net /A5(SCL)(2): track 0.00 -> 7.50 mm
- net /A5(SCL): track 7.50 -> 0.00 mm
- net /Vin: vias 0 -> 1
- net /Reset: vias 2 -> 0
Changed lines of the file:
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@@
     (grid_origin 110.998 126.365)
     (pcbplotparams
-      (layerselection 0x0000030_80000001)
+      (layerselection 0x00010fc_ffffffff)
       (disableapertmacros false)
-      (usegerberextensions false)
-      (usegerberattributes true)
+      (usegerberextensions true)
+      (usegerberattributes false)
       (usegerberadvancedattributes true)
-      (creategerberjobfile true)
+      (creategerberjobfile false)
       (svguseinch false)
       (svgprecision 6)
@@
       (plotinvisibletext false)
       (sketchpadsonfab false)
-      (subtractmaskfromsilk false)
+      (subtractmaskfromsilk true)
       (outputformat 1)
       (mirror false)
-      (drillshape 1)
+      (drillshape 0)
       (scaleselection 1)
-      (outputdirectory "")
+      (outputdirectory "Gerbers")
     )
   )
@@
   (net 52 "Net-(JP1-Pad1)")
   (net 53 "Net-(JP1-Pad2)")
+  (net 54 "/A5(SCL)(2)")
+  (net 55 "/A4(SDA)(2)")
   (footprint "Socket_Arduino_Uno:Socket_Strip_Arduino_1x08" locked (layer "F.Cu")
     (at 138.938 123.825)
@@
     (fp_line (start -1.75 -1.75) (end -1.75 1.75) (layer "F.CrtYd") (width 0.05))
     (pad "1" thru_hole oval locked (at 0 0) (size 1.7272 2.032) (drill 1.016) (layers *.Cu *.Mask "F.SilkS")
-      (net 12 "/A5(SCL)") (pinfunction "Pin_1") (pintype "passive"))
+      (net 54 "/A5(SCL)(2)") (pinfunction "Pin_1") (pintype "passive"))
     (pad "2" thru_hole oval locked (at 2.54 0) (size 1.7272 2.032) (drill 1.016) (layers *.Cu *.Mask "F.SilkS")
-      (net 11 "/A4(SDA)") (pinfunction "Pin_2") (pintype "passive"))
+      (net 55 "/A4(SDA)(2)") (pinfunction "Pin_2") (pintype "passive"))
     (pad "3" thru_hole oval locked (at 5.08 0) (size 1.7272 2.032) (drill 1.016) (layers *.Cu *.Mask "F.SilkS")
       (net 10 "/AREF") (pinfunction "Pin_3") (pintype "passive"))
@@
       (net 3 "+5V") (pintype "passive"))
     (pad "2" smd roundrect (at 0.9125 0) (size 0.975 0.95) (layers "F.Cu" "F.Paste" "F.Mask") (roundrect_rratio 0.25)
-      (net 12 "/A5(SCL)") (pintype "passive"))
+      (net 54 "/A5(SCL)(2)") (pintype "passive"))
     (model "${KICAD6_3DMODEL_DIR}/Resistor_SMD.3dshapes/R_0603_1608Metric.wrl"
       (offset (xyz 0 0 0))
@@
       (net 3 "+5V") (pinfunction "HV") (pintype "power_in"))
     (pad "11" thru_hole oval (at -3.81 -5.08) (size 1.2 2) (drill 0.8) (layers *.Cu *.Mask)
-      (net 11 "/A4(SDA)") (pinfunction "HV2") (pintype "bidirectional"))
+      (net 55 "/A4(SDA)(2)") (pinfunction "HV2") (pintype "bidirectional"))
     (pad "12" thru_hole oval (at -6.35 -5.08) (size 1.2 2) (drill 0.8) (layers *.Cu *.Mask)
-      (net 12 "/A5(SCL)") (pinfunction "HV1") (pintype "bidirectional"))
+      (net 54 "/A5(SCL)(2)") (pinfunction "HV1") (pintype "bidirectional"))
   )
   (footprint "Connector_PinHeader_2.54mm:PinHeader_1x03_P2.54mm_Vertical" (layer "F.Cu")
@@
       (net 4 "GND") (pinfunction "OUT-") (pintype "power_out"))
     (pad "4" thru_hole circle (at 8.5 18) (size 1.7 1.7) (drill 1) (layers *.Cu *.Mask)
-      (net 26 "Net-(J2-Pad2)") (pinfunction "B-") (pintype "unspecified"))
+      (net 26 "Net-(J2-Pad2)") (pinfunction "B-") (pintype "passive"))
     (pad "5" thru_hole circle (at 8.5 8.5) (size 1.7 1.7) (drill 1) (layers *.Cu *.Mask)
-      (net 25 "Net-(J2-Pad1)") (pinfunction "B+") (pintype "bidirectional"))
+      (net 25 "Net-(J2-Pad1)") (pinfunction "B+") (pintype "passive"))
     (pad "6" thru_hole circle (at -11.5 -8) (size 1.7 1.7) (drill 1) (layers *.Cu *.Mask)
       (net 40 "Net-(SW1-Pad2)") (pinfunction "OUT+") (pintype "power_out"))
@@
       (net 3 "+5V") (pintype "passive"))
     (pad "2" smd roundrect (at 0.9125 0 180) (size 0.975 0.95) (layers "F.Cu" "F.Paste" "F.Mask") (roundrect_rratio 0.25)
-      (net 11 "/A4(SDA)") (pintype "passive"))
+      (net 55 "/A4(SDA)(2)") (pintype "passive"))
     (model "${KICAD6_3DMODEL_DIR}/Resistor_SMD.3dshapes/R_0603_1608Metric.wrl"
       (offset (xyz 0 0 0))
@@
     (effects (font (size 1 1) (thickness 0.15)))
   )
+  (segment (start 156.972 110.871) (end 176.164 110.871) (width 0.6) (layer "F.Cu") (net 2))
   (segment (start 176.164 110.871) (end 176.276 110.759) (width 0.6) (layer "F.Cu") (net 2))
-  (segment (start 173.228 110.871) (end 176.164 110.871) (width 0.6) (layer "F.Cu") (net 2))
   (segment (start 144.018 123.825) (end 156.972 110.871) (width 0.6) (layer "F.Cu") (net 2))
-  (via (at 156.972 110.871) (size 0.6) (drill 0.4) (layers "F.Cu" "B.Cu") (net 2))
-  (via (at 173.228 110.871) (size 0.6) (drill 0.4) (layers "F.Cu" "B.Cu") (net 2))
-  (segment (start 156.972 110.871) (end 173.228 110.871) (width 0.6) (layer "B.Cu") (net 2))
-  (segment (start 129.794 121.069498) (end 134.065022 125.34052) (width 0.6) (layer "F.Cu") (net 5))
-  (segment (start 155.20248 125.34052) (end 156.718 123.825) (width 0.6) (layer "F.Cu") (net 5))
-  (segment (start 134.065022 125.34052) (end 155.20248 125.34052) (width 0.6) (layer "F.Cu") (net 5))
-  (segment (start 129.794 121.069498) (end 129.794 90.805) (width 0.6) (layer "F.Cu") (net 5))
-  (segment (start 137.668 80.645) (end 137.5175 80.645) (width 0.6) (layer "F.Cu") (net 11))
-  (segment (start 137.5175 80.645) (end 134.9775 78.105) (width 0.6) (layer "F.Cu") (net 11))
-  (segment (start 132.334 75.565) (end 132.4375 75.565) (width 0.6) (layer "F.Cu") (net 11))
-  (segment (start 132.4375 75.565) (end 134.9775 78.105) (width 0.6) (layer "F.Cu") (net 11))
-  (segment (start 137.414 80.645) (end 137.668 80.645) (width 0.6) (layer "F.Cu") (net 11))
-  (segment (start 129.794 75.6685) (end 132.2305 78.105) (width 0.6) (layer "F.Cu") (net 12))
-  (segment (start 134.7705 80.645) (end 132.2305 78.105) (width 0.6) (layer "F.Cu") (net 12))
-  (segment (start 129.794 75.565) (end 129.794 75.6685) (width 0.6) (layer "F.Cu") (net 12))
-  (segment (start 135.128 80.645) (end 134.7705 80.645) (width 0.6) (layer "F.Cu") (net 12))
+  (segment (start 129.794 90.805) (end 129.794 116.713) (width 0.6) (layer "F.Cu") (net 5))
+  (via (at 129.794 116.713) (size 0.6) (drill 0.4) (layers "F.Cu" "B.Cu") (net 5))
+  (segment (start 129.794 121.069498) (end 134.065022 125.34052) (width 0.6) (layer "B.Cu") (net 5))
+  (segment (start 155.20248 125.34052) (end 156.718 123.825) (width 0.6) (layer "B.Cu") (net 5))
+  (segment (start 134.065022 125.34052) (end 155.20248 125.34052) (width 0.6) (layer "B.Cu") (net 5))
+  (segment (start 129.794 116.713) (end 129.794 121.069498) (width 0.6) (layer "B.Cu") (net 5))
   (segment (start 147.828 77.851) (end 150.114 75.565) (width 0.6) (layer "F.Cu") (net 13))
   (segment (start 147.828 80.645) (end 147.828 77.851) (width 0.6) (layer "F.Cu") (net 13))
@@
   (segment (start 172.1085 100.457) (end 176.164 100.457) (width 0.6) (layer "F.Cu") (net 53))
   (segment (start 176.164 100.457) (end 176.276 100.345) (width 0.6) (layer "F.Cu") (net 53))
+  (segment (start 129.794 75.6685) (end 132.2305 78.105) (width 0.6) (layer "F.Cu") (net 54))
+  (segment (start 134.7705 80.645) (end 132.2305 78.105) (width 0.6) (layer "F.Cu") (net 54))
+  (segment (start 129.794 75.565) (end 129.794 75.6685) (width 0.6) (layer "F.Cu") (net 54))
+  (segment (start 135.128 80.645) (end 134.7705 80.645) (width 0.6) (layer "F.Cu") (net 54))
+  (segment (start 137.668 80.645) (end 137.5175 80.645) (width 0.6) (layer "F.Cu") (net 55))
+  (segment (start 137.5175 80.645) (end 134.9775 78.105) (width 0.6) (layer "F.Cu") (net 55))
+  (segment (start 132.334 75.565) (end 132.4375 75.565) (width 0.6) (layer "F.Cu") (net 55))
+  (segment (start 132.4375 75.565) (end 134.9775 78.105) (width 0.6) (layer "F.Cu") (net 55))
+  (segment (start 137.414 80.645) (end 137.668 80.645) (width 0.6) (layer "F.Cu") (net 55))
   (zone (net 3) (net_name "+5V") (layer "F.Cu") (hatch edge 0.508)
     (connect_pads (clearance 0.508))
