File: Air Bearing PCB/Air_Bearing_PCB.kicad_sch (KiCad schematic)
At the start: 20 parts, among them J1 Conn_01x03_Female, J2 Conn_01x02_Female, J3 Conn_01x06_Female, P1 Power, P2 Analog, P3 Digital, P4 Digital, P5 CONN_01X01, P6 CONN_01X01, P7 CONN_01X01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

Commit message: Added Gerber Files
Made a few small routing and schematic edits. Added Gerber files.
Connections:
- net A4(SDA): no longer P3.2 (Pin_2), R1.2, U2.11 (HV2)
- net A5(SCL): no longer P3.1 (Pin_1), R2.2, U2.12 (HV1)
- new net A4(SDA)(2): P3.2 (Pin_2), R1.2, U2.11 (HV2)
- new net A5(SCL)(2): P3.1 (Pin_1), R2.2, U2.12 (HV1)
Changed lines of the file:
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@@
     (effects (font (size 1.524 1.524)) (justify left bottom))
   )
-  (label "A4(SDA)" (at 267.97 33.02 0)
+  (label "A4(SDA)(2)" (at 267.97 33.02 0)
     (effects (font (size 1.524 1.524)) (justify left bottom))
   )
@@
     (effects (font (size 1.524 1.524)) (justify left bottom))
   )
-  (label "A5(SCL)" (at 111.76 30.48 0)
+  (label "A5(SCL)(2)" (at 111.76 30.48 0)
     (effects (font (size 1.27 1.27)) (justify left bottom))
   )
@@
     (effects (font (size 1.27 1.27)) (justify left bottom))
   )
-  (label "A5(SCL)" (at 267.97 30.48 0)
+  (label "A5(SCL)(2)" (at 267.97 30.48 0)
     (effects (font (size 1.524 1.524)) (justify left bottom))
   )
-  (label "A4(SDA)" (at 111.76 33.02 0)
+  (label "A4(SDA)(2)" (at 111.76 33.02 0)
     (effects (font (size 1.27 1.27)) (justify left bottom))
   )
@@
     (effects (font (size 1.524 1.524)) (justify left bottom))
   )
-  (symbol (lib_id "Connector_Generic:Conn_01x08") (at 243.84 48.26 0) (unit 1)
+  (symbol (lib_name "Conn_01x08_1") (lib_id "Connector_Generic:Conn_01x08") (at 243.84 48.26 0) (unit 1)
     (in_bom yes) (on_board yes)
     (property "Reference" "P1" (id 0) (at 243.84 36.83 0))
